File: usb-c-banana-with-data/usb-c-banana-with-data.kicad_pcb (KiCad board)
At the start: 2 copper layers, 12 parts, among them J1 TYPE-C-31-M-12, J2 Conn_01x01, J3 Conn_01x01, J4 TYPE-C-31-M-12

Commit message: usb-c-banana-with-data: hardware v1.0
Parts:
- moved R4 43.2 mm to (92.8, 115.5)
- moved R5 40.2 mm to (89.5, 102.6), turned to 90 degrees
- moved R3 38.8 mm to (92.8, 103.5)
- moved D1 36.9 mm to (92.0, 101.9), turned to 180 degrees
- moved R6 21.6 mm to (107.8, 101.8)
- moved D2 18.5 mm to (110.3, 102.5), turned to 90 degrees
Routing:
- net VBUS: track 0.00 -> 33.7 mm, vias 0 -> 2
- net GND: track 0.00 -> 27.0 mm, vias 0 -> 27
- net Net-(J4-VBUS-PadA4B9): track 0.00 -> 16.2 mm, vias 0 -> 4
- net Net-(J1-CC2): track 0.00 -> 10.8 mm, vias 0 -> 2
- net Net-(J1-CC1): track 0.00 -> 10.3 mm, vias 0 -> 2
- net Net-(J4-CC1): track 0.00 -> 7.77 mm, vias 0 -> 2
- net Net-(J4-CC2): track 0.00 -> 6.43 mm
- net Net-(D2-A): track 0.00 -> 1.44 mm
- net Net-(D1-A): track 0.00 -> 1.42 mm
- net /D2_P: track 11.7 -> 11.2 mm
- added copper zone on B.Cu, net GND
- added copper zone on F.Cu, net GND
Other:
- board outline added: 24 x 31 mm
- board text added: "DATA"
- board text added: "POWER"
