File: usb-c-banana-with-data/usb-c-banana-with-data.kicad_sch (KiCad schematic)
At the start: 12 parts, among them J1 TYPE-C-31-M-12, J2 Conn_01x01, J3 Conn_01x01, J4 TYPE-C-31-M-12

Commit message: usb-c-banana-with-data: hardware v1.0
Parts:
- J2, J3: LCSC C4994335 -> (none)
Changed lines of the file:
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@@
-			)
-		)
-		(property "LCSC" "C4994335"
-			(at 20.32 58.42 0)
-			(effects
-				(font
-					(size 1.27 1.27)
-				)
-				(hide yes)
 			)
 		)
@@
 			(at 20.32 38.1 0)
 			(effects
-				(font
-					(size 1.27 1.27)
-				)
-				(hide yes)
-			)
-		)
-		(property "LCSC" "C4994335"
-			(at 20.32 38.1 0)
-			(effects
